File: micromouse-pcb/IRsensors.kicad_sch (KiCad schematic)
At the start: 13 parts, among them Q1 BC847, Q2 IRLML0030

Commit message: Finalised schematic
Parts:
- C19: value C_Polarized -> 10uF
- C20: value C -> 100nF
- R10, R15: value R -> 1k
- R11, R16: value R -> 10k
- R12: value R -> 50R
- R13: value R -> 3R3
- R14: value R -> 710mR
Changed lines of the file:
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@@
 			)
 		)
-		(property "Value" "R"
+		(property "Value" "1k"
 			(at 182.88 46.9899 0)
 			(effects
@@
 			)
 		)
-		(property "Value" "R"
+		(property "Value" "50R"
 			(at 78.74 26.67 90)
 			(effects
@@
 			)
 		)
-		(property "Value" "C_Polarized"
+		(property "Value" "10uF"
 			(at 113.03 57.5309 0)
 			(effects
@@
 			)
 		)
-		(property "Value" "C"
+		(property "Value" "100nF"
 			(at 204.47 60.9599 0)
 			(effects
@@
 			)
 		)
-		(property "Value" "R"
+		(property "Value" "10k"
 			(at 53.34 73.6599 0)
 			(effects
@@
 			)
 		)
-		(property "Value" "R"
+		(property "Value" "1k"
 			(at 45.72 54.61 90)
 			(effects
@@
 			)
 		)
-		(property "Value" "R"
+		(property "Value" "3R3"
 			(at 87.63 35.5599 0)
 			(effects
@@
 			)
 		)
-		(property "Value" "R"
+		(property "Value" "10k"
 			(at 182.88 74.9299 0)
 			(effects
@@
 			)
 		)
-		(property "Value" "R"
+		(property "Value" "710mR"
 			(at 87.63 76.1999 0)
 			(effects
