File: micromouse-pcb/micromouse-pcb.kicad_sch (KiCad schematic)
At the start: 28 parts, among them IC1 ICM-42688-P, J3 Conn_01x02_Pin, SW1 SW_MEC_5E, SW2 SW_MEC_5E, U1 AMS1117-3.3, U2 STM32F446RETx, U3 VL53L0CXV0DH1

Commit message: Finalised schematic
Parts:
- added D10: Blue, symbol Device:LED
- added D9: Red, symbol Device:LED
- added J4: Conn_01x06_Socket, symbol Connector:Conn_01x06_Socket
- added J5: Conn_01x05_Socket, symbol Connector:Conn_01x05_Socket
- added R38: 270R, symbol Device:R
- added R39: 20R, symbol Device:R
- added SW3, SW4: SW_MEC_5E, Button_Switch_SMD:SW_Push_1P1T_NO_6x6mm_H9.5mm, symbol Switch:SW_MEC_5E
- C10, C12, C13: value C -> 100nF
- C14, C8: value C -> 1uF
- C3: value C -> 2.2uF
- R4, R5: value R -> 4K7; footprint Resistor_SMD:R_1210_3225Metric -> (none)
Connections:
- net +3.3V: now also C10.1, C12.1, C8.1, IC1.5 (VDDIO), IC1.8 (VDD), R4.2, R5.2, J4.5 (Pin_5), J5.1 (Pin_1), R38.2, R39.1
- net GND: now also C10.2, C12.2, C8.2, IC1.6 (GND), J4.4 (Pin_4), J5.3 (Pin_3), SW3.1, SW3.2, SW4.1, SW4.2
- net VBATT_ADC: now also U2.20 (PA4)
- net ~{RESET}: now also J5.5 (Pin_5)
- net ICM_42688_MISO: now reaches IC1.1 (AP_SDO_/_AP_AD0)
- net ICM_42688_MISO: now also U2.35 (PB14)
- net ICM-42688_CS: now reaches IC1.12 (AP_CS)
- net ICM-42688_CS: now also U2.34 (PB13)
- net ICM-42688_SCK: now reaches IC1.13 (AP_SCL_/_AP_SCLK)
- net ICM-42688_SCK: now also U2.29 (PB10)
- net ICM-42688_MOSI: now reaches IC1.14 (AP_SDA_/_AP_SDIO_/_AP_SDI)
- net ICM-42688_MOSI: now also U2.36 (PB15)
- net ICM-42688_INT1: now reaches IC1.4 (INT1_/_INT)
- net ICM-42688_INT1: now also U2.22 (PA6)
- net ICM_42688_INT2: now reaches IC1.9 (INT2_/_FSYNC_/_CLKIN)
- net ICM_42688_INT2: now also U2.23 (PA7)
- net VL53L4CD_SDA: now reaches R4.1
- net VL53L4CD_SDA: now also U2.61 (PB8), U3.9 (SDA)
- net IR_L: now reaches U2.10 (PC2)
- net IR_R: now reaches U2.11 (PC3)
- net SW1: now reaches U2.14 (PA0)
- net SW1: now also SW3.3 (K), SW3.4 (A)
- net SW2: now reaches U2.15 (PA1)
- net SW2: now also SW4.3 (K), SW4.4 (A)
- net VL53L4CD_INT: now reaches U2.2 (PC13)
- net VL53L4CD_INT: now also U3.7 (GPIO1)
- net IR_Front_L_Pulse: now reaches U2.26 (PB0)
- net IR_Front_R_Pulse: now reaches U2.27 (PB1)
- net IR_L_Pulse: now reaches U2.28 (PB2)
- net VL53L4CD_EN: now reaches U2.3 (PC14)
- net VL53L4CD_EN: now also U3.5 (XSHUT)
- net LMotor_A: now reaches U2.37 (PC6)
- net LMotor_B: now reaches U2.38 (PC7)
- net RMotor_A: now reaches U2.39 (PC8)
- net Motors_EN: now reaches U2.4 (PC15)
- net RMotor_B: now reaches U2.40 (PC9)
- net HC-05_RX: now reaches U2.42 (PA9)
- net HC-05_RX: now also J4.2 (Pin_2)
- net HC-05_TX: now reaches U2.43 (PA10)
- net HC-05_TX: now also J4.3 (Pin_3)
- net SWDIO: now reaches U2.46 (PA13)
- net SWDIO: now also J5.4 (Pin_4)
- net SWDCLK: now reaches U2.49 (PA14)
- net LED1: now reaches U2.5 (PH0)
- net LED1: now also D9.1 (K)
- net IR_R_Pulse: now reaches U2.55 (PB3)
- net L_ENC_A: now reaches U2.56 (PB4)
- net L_ENC_B: now reaches U2.57 (PB5)
- net R_ENC_A: now reaches U2.58 (PB6)
- net R_ENC_B: now reaches U2.59 (PB7)
- net LED2: now reaches U2.6 (PH1)
- net LED2: now also D10.1 (K)
- net VL53L4CD_SCL: now reaches U2.62 (PB9)
- net VL53L4CD_SCL: now also R5.1, U3.10 (SCL)
- net IR_Front_L: now reaches U2.8 (PC0)
- net IR_Front_R: now reaches U2.9 (PC1)
- new net: D9.2 (A), R38.1
- new net: D10.2 (A), R39.2
- new net HC-05_KEY: J4.6 (Pin_6)
- new net HC-05_STATE: J4.1 (Pin_1)
- new net SWCLK: J5.2 (Pin_2)
Other:
- moved on the sheet: C10, C12, C14, C8, IC1

Commit message: Updated schematics and brought in board shape from CAD
Parts:
- removed SW1, SW2, SW3, SW4: SW_MEC_5E, Button_Switch_SMD:SW_Push_1P1T_NO_6x6mm_H9.5mm, symbol Switch:SW_MEC_5E
- added SW1, SW2, SW5, SW6: SW_Push, Button_Switch_SMD:SW_Push_1P1T_NO_CK_KSC6xxJ, symbol Switch:SW_Push
- D10, D9: footprint (none) -> LED_SMD:LED_0603_1608Metric
- F1: footprint Fuse:Fuse_Littelfuse-LVR200 -> Fuse:Fuse_1210_3225Metric
- J4: footprint (none) -> Connector_PinSocket_2.54mm:PinSocket_1x06_P2.54mm_Vertical
- J5: footprint (none) -> Connector_PinHeader_2.54mm:PinHeader_1x05_P2.54mm_Vertical
- R38: footprint (none) -> Resistor_SMD:R_0603_1608Metric_Pad0.98x0.95mm_HandSolder
- R39, R4, R5: footprint (none) -> Resistor_SMD:R_0603_1608Metric
Connections:
- net +3.3V: now also SW5.1
- net GND: now also SW1.1, SW2.1, SW6.1
- net SW1: now also SW1.2
- net SW2: now also SW2.2
- net ~{RESET}: now also SW6.2
- net at R3.1: now also SW5.2
