File: micromouse-pcb/motor-driver.kicad_sch (KiCad schematic)
At the start: 10 parts, among them J1 Conn_01x06_Socket, J2 Conn_01x06_Socket, U4 DRV8833RTY

Commit message: Finalised schematic
Parts:
- C17: value C -> 100nF
- C18: value C_Polarized -> 10uF
- R7, R8: value R -> 10R
- R9: value R -> 10K
Changed lines of the file:
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@@
 			)
 		)
-		(property "Value" "R"
+		(property "Value" "10K"
 			(at 198.12 76.1999 0)
 			(effects
@@
 			)
 		)
-		(property "Value" "R"
+		(property "Value" "10R"
 			(at 115.57 91.4399 0)
 			(effects
@@
 			)
 		)
-		(property "Value" "C_Polarized"
+		(property "Value" "10uF"
 			(at 180.34 74.0409 0)
 			(effects
@@
 			)
 		)
-		(property "Value" "R"
+		(property "Value" "10R"
 			(at 106.68 91.4399 0)
 			(effects
@@
 			)
 		)
-		(property "Value" "C"
+		(property "Value" "100nF"
 			(at 167.64 74.9299 0)
 			(effects
