File: micromouse-pcb/micromouse-pcb.kicad_pcb (KiCad board)
At the start: 2 copper layers, 110 x 110 mm, 90 parts, among them IC1 ICM-42688-P, J1 Conn_01x06_Socket, J2 Conn_01x06_Socket, J3 Conn_01x02_Pin, Q1 BC847, Q2 IRLML0030, Q3 BC847, Q4 IRLML0030, Q5 BC847, Q6 IRLML0030, Q7 BC847, Q8 IRLML0030, SW1 SW_MEC_5E, SW2 SW_MEC_5E, U1 AMS1117-3.3, U2 STM32F446RETx, U3 VL53L0CXV0DH1, U4 DRV8833RTY

Commit message: Updated schematics and brought in board shape from CAD
Parts:
- added D10: Blue, LED_SMD:LED_0603_1608Metric, F.Cu at (182.0, 50.7)
- added D9: Red, LED_SMD:LED_0603_1608Metric, F.Cu at (182.0, 48.1)
- added J4: Conn_01x06_Socket, Connector_PinSocket_2.54mm:PinSocket_1x06_P2.54mm_Vertical, F.Cu at (112.0, 85.6)
- added J5: Conn_01x05_Socket, Connector_PinHeader_2.54mm:PinHeader_1x05_P2.54mm_Vertical, F.Cu at (79.0, 85.6)
- added R38: 270R, Resistor_SMD:R_0603_1608Metric_Pad0.98x0.95mm_HandSolder, F.Cu at (186.2, 48.1)
- added R39: 20R, Resistor_SMD:R_0603_1608Metric, F.Cu at (178.0, 53.1)
- added SW5: SW_Push, Button_Switch_SMD:SW_Push_1P1T_NO_CK_KSC6xxJ, F.Cu at (120.0, 138.0)
- added SW6: SW_Push, Button_Switch_SMD:SW_Push_1P1T_NO_CK_KSC6xxJ, F.Cu at (119.0, 131.0)
- C10, C12, C13, C17, C20, C22, C24, C26: value C -> 100nF
- C14, C8: value C -> 1uF
- C18, C19, C21, C23, C25: value C_Polarized -> 10uF
- C3: value C -> 2.2uF
- F1: footprint Fuse:Fuse_Littelfuse-LVR200 -> Fuse:Fuse_1210_3225Metric
- R10, R15, R17, R22, R24, R29, R31, R36: value R -> 1k
- R11, R16, R18, R23, R25, R30, R32, R37: value R -> 10k
- R12, R19, R26, R33: value R -> 50R
- R13, R20, R27, R34: value R -> 3R3
- R14, R21, R28, R35: value R -> 710mR
- R4, R5: value R -> 4K7; footprint Resistor_SMD:R_1210_3225Metric -> Resistor_SMD:R_0603_1608Metric
- R7, R8: value R -> 10R
- R9: value R -> 10K
- SW1, SW2: value SW_MEC_5E -> SW_Push; footprint Button_Switch_SMD:SW_Push_1P1T_NO_6x6mm_H9.5mm -> Button_Switch_SMD:SW_Push_1P1T_NO_CK_KSC6xxJ
- moved J1 141.4 mm to (80.0, 123.0), turned to -90 degrees
- moved U4 136.1 mm to (93.0, 127.1), turned to 90 degrees
- moved C18 130.9 mm to (93.7, 136.0)
- moved SW1 125.7 mm to (68.0, 136.0)
- moved C25 120.6 mm to (99.0, 65.0)
- moved C23 120.5 mm to (65.0, 85.0)
- moved C16 120.4 mm to (93.0, 121.0)
- moved D2 119.5 mm to (104.0, 154.0)
- moved D4 116.7 mm to (80.5, 154.0)
- moved SW2 116.7 mm to (68.0, 126.0)
- moved J2 115.7 mm to (106.0, 122.5), turned to -90 degrees
- moved IC1 111.3 mm to (95.0, 103.1)
- moved D1 109.4 mm to (104.0, 146.0)
- moved D3 106.6 mm to (80.5, 146.0)
- moved D8 102.6 mm to (114.0, 154.0)
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Connections:
- C10 pad 1: unconnected-(C10-Pad1) -> +3.3V
- C10 pad 2: unconnected-(C10-Pad2) -> GND
- C12 pad 1: unconnected-(C12-Pad1) -> +3.3V
- C12 pad 2: unconnected-(C12-Pad2) -> GND
- C8 pad 1: unconnected-(C8-Pad1) -> +3.3V
- C8 pad 2: unconnected-(C8-Pad2) -> GND
- D2 pad 2: /Front Right/Sense -> /IR_Front_R
- D4 pad 2: /Left/Sense -> /IR_L
- D6 pad 2: /Front Left/Sense -> /IR_Front_L
- D8 pad 2: /Right/Sense -> /IR_R
- IC1 pad 1: unconnected-(IC1-AP_SDO_/_AP_AD0-Pad1) -> /ICM_42688_MISO
- IC1 pad 12: unconnected-(IC1-AP_CS-Pad12) -> /ICM-42688_CS
- IC1 pad 13: unconnected-(IC1-AP_SCL_/_AP_SCLK-Pad13) -> /ICM-42688_SCK
- IC1 pad 14: unconnected-(IC1-AP_SDA_/_AP_SDIO_/_AP_SDI-Pad14) -> /ICM-42688_MOSI
- IC1 pad 4: unconnected-(IC1-INT1_/_INT-Pad4) -> /ICM-42688_INT1
- IC1 pad 5: unconnected-(IC1-VDDIO-Pad5) -> +3.3V
- IC1 pad 6: unconnected-(IC1-GND-Pad6) -> GND
- IC1 pad 8: unconnected-(IC1-VDD-Pad8) -> +3.3V
- IC1 pad 9: unconnected-(IC1-INT2_/_FSYNC_/_CLKIN-Pad9) -> /ICM_42688_INT2
- J1 pad 3: /Motor Driver/LMotorEncA -> /R_ENC_A
- J1 pad 4: /Motor Driver/LMotorEncB -> /R_ENC_B
- J2 pad 3: /Motor Driver/RMotorEncA -> /L_ENC_B
- J2 pad 4: /Motor Driver/RMotorEncB -> /L_ENC_A
- R10 pad 1: /Front Right/IR_Pulse -> /IR_Front_R_Pulse
- R16 pad 1: /Front Right/Sense -> /IR_Front_R
- R17 pad 1: /Left/IR_Pulse -> /IR_L_Pulse
- R23 pad 1: /Left/Sense -> /IR_L
- R24 pad 1: /Front Left/IR_Pulse -> /IR_Front_L_Pulse
- R30 pad 1: /Front Left/Sense -> /IR_Front_L
- R31 pad 1: /Right/IR_Pulse -> /IR_R_Pulse
- R37 pad 1: /Right/Sense -> /IR_R
- R4 pad 1: unconnected-(R4-Pad1) -> /VL53L4CD_SDA
- R4 pad 2: unconnected-(R4-Pad2) -> +3.3V
- R5 pad 1: unconnected-(R5-Pad1) -> /VL53L4CD_SCL
- R5 pad 2: unconnected-(R5-Pad2) -> +3.3V
- SW1 pad 1: +3.3V -> GND
- SW1 pad 2: +3.3V -> /SW1
- SW2 pad 2: GND -> /SW2
- U2 pad 10: unconnected-(U2-PC2-Pad10) -> /IR_L
- U2 pad 11: unconnected-(U2-PC3-Pad11) -> /IR_R
- U2 pad 14: unconnected-(U2-PA0-Pad14) -> /SW1
- U2 pad 15: unconnected-(U2-PA1-Pad15) -> /SW2
- U2 pad 2: unconnected-(U2-PC13-Pad2) -> /VL53L4CD_INT
- U2 pad 20: unconnected-(U2-PA4-Pad20) -> /VBATT_ADC
- U2 pad 22: unconnected-(U2-PA6-Pad22) -> /ICM-42688_INT1
- U2 pad 23: unconnected-(U2-PA7-Pad23) -> /ICM_42688_INT2
- U2 pad 26: unconnected-(U2-PB0-Pad26) -> /IR_Front_L_Pulse
- U2 pad 27: unconnected-(U2-PB1-Pad27) -> /IR_Front_R_Pulse
- U2 pad 28: unconnected-(U2-PB2-Pad28) -> /IR_L_Pulse
- U2 pad 29: unconnected-(U2-PB10-Pad29) -> /ICM-42688_SCK
- U2 pad 3: unconnected-(U2-PC14-Pad3) -> /VL53L4CD_EN
- U2 pad 34: unconnected-(U2-PB13-Pad34) -> /ICM-42688_CS
- U2 pad 35: unconnected-(U2-PB14-Pad35) -> /ICM_42688_MISO
- U2 pad 36: unconnected-(U2-PB15-Pad36) -> /ICM-42688_MOSI
- U2 pad 37: unconnected-(U2-PC6-Pad37) -> /LMotor_A
- U2 pad 38: unconnected-(U2-PC7-Pad38) -> /LMotor_B
- U2 pad 39: unconnected-(U2-PC8-Pad39) -> /RMotor_A
- U2 pad 4: unconnected-(U2-PC15-Pad4) -> /Motors_EN
- U2 pad 40: unconnected-(U2-PC9-Pad40) -> /RMotor_B
- U2 pad 42: unconnected-(U2-PA9-Pad42) -> /HC-05_RX
- U2 pad 43: unconnected-(U2-PA10-Pad43) -> /HC-05_TX
- U2 pad 46: unconnected-(U2-PA13-Pad46) -> /SWDIO
- U2 pad 49: unconnected-(U2-PA14-Pad49) -> /SWDCLK
- U2 pad 5: unconnected-(U2-PH0-Pad5) -> /LED1
- U2 pad 55: unconnected-(U2-PB3-Pad55) -> /IR_R_Pulse
- U2 pad 56: unconnected-(U2-PB4-Pad56) -> /L_ENC_A
- U2 pad 57: unconnected-(U2-PB5-Pad57) -> /L_ENC_B
- U2 pad 58: unconnected-(U2-PB6-Pad58) -> /R_ENC_A
- U2 pad 59: unconnected-(U2-PB7-Pad59) -> /R_ENC_B
- U2 pad 6: unconnected-(U2-PH1-Pad6) -> /LED2
- U2 pad 61: unconnected-(U2-PB8-Pad61) -> /VL53L4CD_SDA
- U2 pad 62: unconnected-(U2-PB9-Pad62) -> /VL53L4CD_SCL
- U2 pad 8: unconnected-(U2-PC0-Pad8) -> /IR_Front_L
- U2 pad 9: unconnected-(U2-PC1-Pad9) -> /IR_Front_R
- U3 pad 10: unconnected-(U3-SCL-Pad10) -> /VL53L4CD_SCL
- U3 pad 5: unconnected-(U3-XSHUT-Pad5) -> /VL53L4CD_EN
- U3 pad 7: unconnected-(U3-GPIO1-Pad7) -> /VL53L4CD_INT
- U3 pad 9: unconnected-(U3-SDA-Pad9) -> /VL53L4CD_SDA
- U4 pad 13: /Motor Driver/LMotor2 -> /LMotor_B
- U4 pad 14: /Motor Driver/LMotor1 -> /LMotor_A
- U4 pad 15: /Motor Driver/Motor_EN -> /Motors_EN
- U4 pad 7: /Motor Driver/RMotor1 -> /RMotor_A
- U4 pad 8: /Motor Driver/RMotor2 -> /RMotor_B
Routing:
- net /SWDIO: track 0.00 -> 32.3 mm, vias 0 -> 1
- net /~{RESET}: track 0.00 -> 12.5 mm
Other:
- board size 110 x 110 mm -> 80 x 117.3 mm

Commit message: Updated outline and PCB file
Parts:
- moved U3 104.8 mm to (72.0, 149.2)
- moved C14 103.1 mm to (72.0, 146.0)
- moved F1 80.7 mm to (112.0, 118.4), turned to -90 degrees
- moved C10 19.8 mm to (149.9, 90.0)
- moved IC1 13.2 mm to (95.0, 89.9)
- moved SW2 5.00 mm to (68.0, 131.0)
- moved C23 3.16 mm to (68.0, 84.0), turned to -90 degrees
- moved SW1 2.00 mm to (68.0, 138.0)
- moved U1 1.19 mm to (120.0, 121.0)
- moved C19 1.00 mm to (121.0, 84.0), turned to -90 degrees
- moved J3 1.00 mm to (118.5, 112.0)
- moved SW5 1.00 mm to (119.0, 138.0)
Routing:
- net /SWDIO: track 32.3 -> 0.00 mm, vias 1 -> 0
- net /~{RESET}: track 12.5 -> 0.00 mm
Other:
- outline, holes or cut-outs redrawn
